File: Base Module/BasePCB/_autosave-BasePCB.kicad_sch (KiCad schematic)
At the start: 146 parts, among them J1 USB_A, J2 Conn_01x05_Female, J3 Conn_01x05_Male, J4 Conn_01x05_Female, J5 Conn_01x05_Female, SW1 SW_Push, U1 ATmega32U4-A, Y1 Crystal_GND24_Small

Commit message: Finished wiring
Other:
- note added: "USB-A"
- note removed: "USB-C"
Changed lines of the file:
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@@
     (stroke (width 0) (type default) (color 0 0 0 0))
   )
-  (text "USB-C" (at 215.9 210.82 0)
+  (text "USB-A\n" (at 215.9 210.82 0)
     (effects (font (size 2.5 2.5) bold) (justify left bottom))
   )
