File: Base Module/BasePCB/BasePCB.kicad_pcb (KiCad board)
At the start: 2 copper layers, 321.5 x 98.4 mm, 146 parts, among them J1 USB_A, J2 Conn_01x05_Female, J3 Conn_01x05_Male, J4 Conn_01x05_Female, J5 Conn_01x05_Female, SW1 SW_Push, U1 ATmega32U4-A, Y1 Crystal_GND24_Small

Commit message: Finished wiring
Routing:
- net VCC: track 64.3 -> 415.3 mm, vias 2 -> 8
- net GND: track 371.4 -> 690.9 mm, vias 8 -> 14
- net +5V: track 306.3 -> 602.1 mm, vias 4 -> 15
- net IN: track 0.00 -> 291.5 mm, vias 0 -> 28
- net OUT: track 163.9 -> 350.1 mm, vias 5 -> 13
- net Net-(J5-Pad3): track 0.00 -> 3.24 mm

Commit message: idk what I did but almost fucked shit up
fixed it I hope
Routing:
- net COL3: track 319.6 -> 317.1 mm
Changed lines of the file:
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@@
   (segment (start -131.191 -92.837) (end -131.191 -85.6975) (width 0.254) (layer "B.Cu") (net 97))
   (segment (start -129.159 -44.1605) (end -53.2485 -44.1605) (width 0.254) (layer "F.Cu") (net 98))
-  (segment (start -14.12875 -54.9275) (end 19.20875 -54.9275) (width 0.254) (layer "F.Cu") (net 98))
   (segment (start -30.7975 -88.4555) (end -30.7975 -88.265) (width 0.254) (layer "F.Cu") (net 98))
   (segment (start -132.08 -96.393) (end -132.08 -94.107) (width 0.254) (layer "F.Cu") (net 98))
@@
   (segment (start -34.925 -107.15625) (end -30.95625 -107.15625) (width 0.254) (layer "F.Cu") (net 98))
   (segment (start -30.95625 -107.15625) (end -29.4875 -105.6875) (width 0.254) (layer "F.Cu") (net 98))
+  (segment (start -21.2725 -56.1975) (end -21.2725 -62.07125) (width 0.254) (layer "F.Cu") (net 98))
   (segment (start -30.7975 -84.8995) (end -30.7975 -88.4555) (width 0.254) (layer "F.Cu") (net 98))
   (segment (start -50.8 -44.196) (end -21.59 -44.196) (width 0.254) (layer "F.Cu") (net 98))
@@
   (segment (start -130.86675 -97.60625) (end -132.08 -96.393) (width 0.254) (layer "F.Cu") (net 98))
   (segment (start -29.4875 -105.6875) (end -29.4875 -94.4875) (width 0.254) (layer "F.Cu") (net 98))
-  (segment (start -21.2725 -44.5135) (end -21.2725 -62.07125) (width 0.254) (layer "F.Cu") (net 98))
+  (segment (start -21.2725 -44.5135) (end -21.2725 -56.1975) (width 0.254) (layer "F.Cu") (net 98))
   (segment (start -34.25 -123.94375) (end -34.25 -113.5375) (width 0.254) (layer "F.Cu") (net 98))
   (segment (start -132.08 -84.709) (end -132.08 -45.72) (width 0.254) (layer "F.Cu") (net 98))
+  (segment (start -20.0025 -54.9275) (end -21.2725 -56.1975) (width 0.254) (layer "F.Cu") (net 98))
   (segment (start -36.5125 -126.20625) (end -34.25 -123.94375) (width 0.254) (layer "F.Cu") (net 98))
   (segment (start -29.464 -83.566) (end -30.7975 -84.8995) (width 0.254) (layer "F.Cu") (net 98))
   (segment (start -21.59 -44.196) (end -21.2725 -44.5135) (width 0.254) (layer "F.Cu") (net 98))
+  (segment (start 19.20875 -54.9275) (end -20.0025 -54.9275) (width 0.254) (layer "F.Cu") (net 98))
   (segment (start -21.2725 -73.9775) (end -21.2725 -81.5975) (width 0.254) (layer "F.Cu") (net 98))
   (segment (start -44.45 -126.20625) (end -36.5125 -126.20625) (width 0.254) (layer "F.Cu") (net 98))
-  (segment (start -21.2725 -62.07125) (end -14.12875 -54.9275) (width 0.254) (layer "F.Cu") (net 98))
   (via (at -132.08 -45.72) (size 0.8) (drill 0.4) (layers "F.Cu" "B.Cu") (net 98))
   (via (at -129.159 -44.1605) (size 0.8) (drill 0.4) (layers "F.Cu" "B.Cu") (net 98))

Commit message: Continued wiring pcb
Parts:
- removed J5: Conn_01x05_Female, Connector_JST:JST_PH_S5B-PH-K_1x05_P2.00mm_Horizontal
- removed R5, R6, R7, R8: 100, Resistor_SMD:R_0805_2012Metric
- J2: value Conn_01x05_Female -> Conn_01x19_Female; footprint Connector_JST:JST_PH_S5B-PH-K_1x05_P2.00mm_Horizontal -> Connector_JST:JST_SH_SM20B-SRSS-TB_1x20-1MP_P1.00mm_Horizontal
- J3: value Conn_01x05_Male -> Conn_01x19_Male; footprint Connector_JST:JST_PH_S5B-PH-K_1x05_P2.00mm_Horizontal -> Connector_JST:JST_SH_SM20B-SRSS-TB_1x20-1MP_P1.00mm_Horizontal
- J4: value Conn_01x05_Female -> Conn_01x18_Female; footprint Connector_JST:JST_PH_S5B-PH-K_1x05_P2.00mm_Horizontal -> Connector_JST:JST_SH_SM20B-SRSS-TB_1x20-1MP_P1.00mm_Horizontal
- moved J4 4.26 mm to (23.0, -138.1), turned to 0 degrees
- moved J2 4.07 mm to (-142.9, -90.5), turned to 90 degrees
- moved J3 4.02 mm to (172.7, -90.5), turned to -90 degrees
Connections:
- J2 pad 3: Net-(J2-Pad3) -> COL0
- J2 pad 4: unconnected-(J2-Pad4) -> COL1
- J2 pad 5: GND -> COL2
- J3 pad 3: Net-(J3-Pad3) -> COL0
- J3 pad 4: unconnected-(J3-Pad4) -> COL1
- J3 pad 5: GND -> COL2
- J4 pad 3: Net-(J4-Pad3) -> COL0
- J4 pad 4: unconnected-(J4-Pad4) -> COL1
- J4 pad 5: GND -> COL2
- U1 pad 1: unconnected-(U1-Pad1) -> ROW10
- U1 pad 31: IN -> ROW8
- U1 pad 32: OUT -> ROW9
- U1 pad 36: unconnected-(U1-Pad36) -> ROW7
- U1 pad 37: unconnected-(U1-Pad37) -> ROW6
- U1 pad 38: unconnected-(U1-Pad38) -> ROW5
Routing:
- net GND: track 690.9 -> 297.4 mm, vias 14 -> 7
- net OUT: track 350.1 -> 0.00 mm, vias 13 -> 0
- net ROW8: track 0.00 -> 304.9 mm, vias 0 -> 32
- net IN: track 291.5 -> 0.00 mm, vias 28 -> 0
- net COL0: track 132.9 -> 401.9 mm, vias 2 -> 32
- net COL1: track 178.1 -> 421.4 mm, vias 2 -> 24
- net COL2: track 249.6 -> 480.3 mm, vias 2 -> 28
- net COL3: track 317.1 -> 507.6 mm, vias 6 -> 17
- net ROW9: track 0.00 -> 160.4 mm, vias 0 -> 5
- net COL4: track 394.5 -> 510.9 mm, vias 10 -> 22
- net COL8: track 339.4 -> 451.0 mm, vias 7 -> 15
- net COL9: track 359.8 -> 469.8 mm, vias 17 -> 19
- net COL5: track 421.5 -> 511.4 mm, vias 14 -> 20
- net COL10: track 380.9 -> 467.3 mm, vias 14 -> 17
- net COL6: track 363.8 -> 429.5 mm, vias 2 -> 6
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Other:
- board size 321.5 x 98.4 mm -> 322.1 x 316.7 mm

Commit message: Continued wiring pcb again
Routing:
- net GND: track 297.4 -> 620.8 mm, vias 7 -> 32
- net COL1: track 421.4 -> 499.2 mm, vias 24 -> 28
- net COL0: track 401.9 -> 476.7 mm, vias 32 -> 36
- net ROW8: track 304.9 -> 379.4 mm, vias 32 -> 35
- net COL10: track 467.3 -> 536.5 mm, vias 17 -> 21
- net COL9: track 469.8 -> 537.7 mm, vias 19 -> 25
- net COL8: track 451.0 -> 517.5 mm, vias 15 -> 22
- net COL6: track 429.5 -> 492.9 mm, vias 6 -> 11
- net ROW9: track 160.4 -> 209.4 mm, vias 5 -> 10
- net ROW5: track 3.20 -> 46.1 mm, vias 0 -> 4
- net ROW7: track 3.05 -> 43.6 mm, vias 0 -> 5
- net ROW6: track 2.82 -> 41.0 mm, vias 0 -> 4
- net VCC: track 378.0 -> 414.6 mm, vias 9 -> 12
- net COL7: track 424.7 -> 458.5 mm, vias 16 -> 19
- net COL2: track 480.3 -> 510.7 mm, vias 28 -> 30
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
Commit message: Finished wiring, added grounded layer
Routing:
- net ROW7: track 43.6 -> 368.3 mm, vias 5 -> 37
- net ROW5: track 46.1 -> 365.2 mm, vias 4 -> 40
- net ROW6: track 41.0 -> 340.9 mm, vias 4 -> 32
- net ROW10: track 1.38 -> 200.8 mm, vias 0 -> 5
- net ROW9: track 209.4 -> 383.0 mm, vias 10 -> 39
- net COL10: track 536.5 -> 624.5 mm, vias 21 -> 25
- net COL3: track 536.6 -> 609.7 mm, vias 19 -> 21
- net COL9: track 537.7 -> 608.1 mm, vias 25 -> 29
- net COL2: track 510.7 -> 574.2 mm, vias 30 -> 35
- net COL8: track 517.5 -> 569.8 mm, vias 22 -> 27
- net COL4: track 524.0 -> 576.1 mm, vias 22 -> 24
- net COL0: track 476.7 -> 519.2 mm, vias 36 -> 43
- net COL1: track 499.2 -> 540.7 mm, vias 28 -> 36
- net COL5: track 523.4 -> 553.5 mm, vias 21 -> 23
- net GND: track 620.8 -> 650.4 mm, vias 32 -> 33
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- added copper zone on B.Cu, net GND

Commit message: Fixed a few errors
Routing:
- net unconnected-(J1-Pad5): track 0.00 -> 14.0 mm

Commit message: Finished PCB
For now
Other:
- board size 322.1 x 316.7 mm -> 321.5 x 98.4 mm
Changed lines of the file:
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@@
     (property "Sheetname" "")
     (attr smd)
-    (fp_text reference "J4" (at 170.6485 -55.7845 90) (layer "F.SilkS")
+    (fp_text reference "J4" (at 0.00775 0.79375 90) (layer "F.SilkS")
       (effects (font (size 1 1) (thickness 0.15)))
     )
@@
   (gr_line (start 175.41875 -135.73125) (end 175.41875 -138.90625) (layer "Edge.Cuts") (width 0.15))
   (gr_line (start -146.05 -135.73125) (end -146.05 -138.90625) (layer "Edge.Cuts") (width 0.15))
-  (gr_line (start -146.633 -240.514) (end -146.633 76.19225) (layer "Edge.Cuts") (width 0.15))
   (gr_arc (start 175.41875 -45.24375) (mid 174.721298 -43.559952) (end 173.0375 -42.8625) (layer "Edge.Cuts") (width 0.15))
   (gr_arc (start 173.0375 -141.2875) (mid 174.721298 -140.590048) (end 175.41875 -138.90625) (layer "Edge.Cuts") (width 0.15))
