File: Base Module/BasePCB/BasePCB.kicad_pcb (KiCad board)
At the start: 2 copper layers, 321.5 x 98.4 mm, 141 parts, among them J1 USB_A, J2 Conn_01x19_Female, J3 Conn_01x19_Male, J4 Conn_01x18_Female, SW1 SW_Push, U1 ATmega32U4-A, Y1 Crystal_GND24_Small

Commit message: Updated conenctors
Parts:
- J2: value Conn_01x19_Female -> Conn_02x10_Counter_Clockwise; footprint Connector_JST:JST_SH_SM20B-SRSS-TB_1x20-1MP_P1.00mm_Horizontal -> Connector_PinSocket_2.54mm:PinSocket_2x10_P2.54mm_Horizontal
- J3: value Conn_01x19_Male -> Conn_02x10_Counter_Clockwise; footprint Connector_JST:JST_SH_SM20B-SRSS-TB_1x20-1MP_P1.00mm_Horizontal -> Connector_PinSocket_2.54mm:PinSocket_2x10_P2.54mm_Horizontal
- J4: value Conn_01x18_Female -> Conn_02x10_Counter_Clockwise; footprint Connector_JST:JST_SH_SM20B-SRSS-TB_1x20-1MP_P1.00mm_Horizontal -> Connector_PinHeader_2.54mm:PinHeader_2x10_P2.54mm_Horizontal
- moved J4 162.7 mm to (181.7, -101.9)
- moved J3 148.1 mm to (34.4, -143.7)
- moved J2 13.5 mm to (-149.9, -101.9), turned to 0 degrees
Connections:
- J2 pad 20: (no net) -> unconnected-(J2-Pad20)
- J3 pad 14: ROW5 -> COL11
- J3 pad 15: ROW6 -> COL12
- J3 pad 16: ROW7 -> COL13
- J3 pad 17: ROW8 -> ROW10
- J3 pad 18: ROW9 -> GND
- J3 pad 19: GND -> unconnected-(J3-Pad19)
- J3 pad 20: (no net) -> unconnected-(J3-Pad20)
- J4 pad 14: COL11 -> ROW5
- J4 pad 15: COL12 -> ROW6
- J4 pad 16: COL13 -> ROW7
- J4 pad 17: ROW10 -> ROW8
- J4 pad 18: GND -> ROW9
- J4 pad 19: (no net) -> GND
- J4 pad 20: (no net) -> unconnected-(J4-Pad20)
Routing:
- net COL0: track 519.1 -> 1010.5 mm, vias 43 -> 79
- net COL1: track 540.7 -> 60.0 mm, vias 36 -> 0
- net ROW10: track 200.8 -> 169.5 mm, vias 5 -> 4
- net GND: track 650.4 -> 628.4 mm, vias 33 -> 29
- net ROW9: track 383.0 -> 396.4 mm
- net ROW7: track 368.1 -> 380.6 mm
- net ROW5: track 365.2 -> 377.1 mm
- net VCC: track 424.0 -> 435.8 mm
- net COL9: track 608.1 -> 619.8 mm
- net COL3: track 609.7 -> 620.7 mm
- net COL7: track 473.7 -> 484.6 mm
- net COL5: track 553.5 -> 564.2 mm
- net ROW8: track 379.4 -> 388.3 mm
- net ROW6: track 340.9 -> 349.4 mm
- net COL10: track 624.5 -> 632.5 mm
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
Commit message: Finished new connectors
Parts:
- moved J1 6.35 mm to (-127.8, -143.1)
Routing:
- net COL1: track 60.0 -> 600.8 mm, vias 0 -> 37
- net COL0: track 1010.5 -> 525.0 mm, vias 79 -> 39
- net VCC: track 435.8 -> 598.1 mm, vias 13 -> 8
- net GND: track 628.4 -> 671.4 mm, vias 29 -> 32
- net ROW9: track 396.4 -> 422.2 mm, vias 39 -> 38
- net COL5: track 564.2 -> 587.9 mm, vias 23 -> 22
- net ROW7: track 380.6 -> 401.2 mm, vias 37 -> 36
- net ROW8: track 388.3 -> 408.7 mm
- net ROW5: track 377.1 -> 393.9 mm, vias 40 -> 37
- net COL4: track 583.2 -> 599.2 mm, vias 24 -> 25
- net ROW6: track 349.4 -> 364.9 mm, vias 32 -> 29
- net COL7: track 484.6 -> 498.3 mm
- net COL3: track 620.7 -> 634.2 mm
- net COL9: track 619.8 -> 631.7 mm, vias 29 -> 26
- net COL11: track 357.9 -> 368.8 mm
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- added copper zone on B.Cu, net (none)
- removed copper zone on B.Cu, net GND
Other:
- board size 321.5 x 98.4 mm -> 339.7 x 104.8 mm

Commit message: Updated mounting holes
Routing:
- added copper zone on B.Cu, net GND
- removed copper zone on B.Cu, net (none)
Other:
- outline, holes or cut-outs redrawn
Changed lines of the file:
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@@
   )
   (gr_line (start -153.9875 -45.24375) (end -153.9875 -145.25625) (layer "Edge.Cuts") (width 0.15))
-  (gr_circle (center -30.1625 -53.975) (end -30.1625 -55.5625) (layer "Edge.Cuts") (width 0.1) (fill none))
+  (gr_circle (center -30.1625 -53.975) (end -30.1625 -54.76875) (layer "Edge.Cuts") (width 0.1) (fill none))
   (gr_arc (start 185.7375 -45.24375) (mid 185.040048 -43.559952) (end 183.35625 -42.8625) (layer "Edge.Cuts") (width 0.15))
   (gr_arc (start 183.35625 -147.6375) (mid 185.040048 -146.940048) (end 185.7375 -145.25625) (layer "Edge.Cuts") (width 0.15))
+  (gr_circle (center -149.225 -143.66875) (end -149.225 -144.4625) (layer "Edge.Cuts") (width 0.1) (fill none))
   (gr_line (start 183.35625 -42.8625) (end -151.60625 -42.8625) (layer "Edge.Cuts") (width 0.15))
-  (gr_circle (center -98.425 -143.66875) (end -98.425 -145.25625) (layer "Edge.Cuts") (width 0.1) (fill none))
-  (gr_line (start 175.41875 -135.73125) (end 175.41875 -138.90625) (layer "Edge.Cuts") (width 0.15))
   (gr_arc (start -151.60625 -42.8625) (mid -153.290048 -43.559952) (end -153.9875 -45.24375) (layer "Edge.Cuts") (width 0.15))
   (gr_line (start 183.35625 -147.6375) (end -151.60625 -147.6375) (layer "Edge.Cuts") (width 0.15))
-  (gr_circle (center 53.18125 -53.975) (end 53.18125 -55.5625) (layer "Edge.Cuts") (width 0.1) (fill none))
-  (gr_circle (center -41.275 -143.66875) (end -40.48125 -145.25625) (layer "Edge.Cuts") (width 0.1) (fill none))
-  (gr_circle (center -150.01875 -143.66875) (end -148.43125 -143.66875) (layer "Edge.Cuts") (width 0.1) (fill none))
-  (gr_circle (center 181.76875 -46.83125) (end 183.35625 -46.83125) (layer "Edge.Cuts") (width 0.1) (fill none))
+  (gr_circle (center 53.18125 -53.975) (end 53.18125 -54.76875) (layer "Edge.Cuts") (width 0.1) (fill none))
+  (gr_circle (center -41.275 -143.66875) (end -41.275 -144.4625) (layer "Edge.Cuts") (width 0.1) (fill none))
+  (gr_circle (center 181.76875 -46.83125) (end 182.5625 -46.83125) (layer "Edge.Cuts") (width 0.1) (fill none))
   (gr_circle (center 181.76875 -46.83125) (end 181.76875 -46.83125) (layer "Edge.Cuts") (width 0.1) (fill none))
-  (gr_arc (start 173.0375 -141.2875) (mid 174.721298 -140.590048) (end 175.41875 -138.90625) (layer "Edge.Cuts") (width 0.15))
-  (gr_circle (center 144.4625 -90.4875) (end 144.4625 -92.075) (layer "Edge.Cuts") (width 0.1) (fill none))
+  (gr_circle (center -98.425 -143.66875) (end -98.425 -144.4625) (layer "Edge.Cuts") (width 0.1) (fill none))
+  (gr_circle (center 144.4625 -90.4875) (end 144.4625 -91.28125) (layer "Edge.Cuts") (width 0.1) (fill none))
   (gr_arc (start -153.9875 -145.25625) (mid -153.290048 -146.940048) (end -151.60625 -147.6375) (layer "Edge.Cuts") (width 0.15))
   (gr_line (start 185.7375 -45.24375) (end 185.7375 -145.25625) (layer "Edge.Cuts") (width 0.15))
-  (gr_circle (center -3.175 -143.66875) (end -1.5875 -143.66875) (layer "Edge.Cuts") (width 0.1) (fill none))
-  (gr_circle (center 145.25625 -128.5875) (end 145.25625 -130.175) (layer "Edge.Cuts") (width 0.1) (fill none))
-  (gr_circle (center -150.01875 -46.83125) (end -150.01875 -48.41875) (layer "Edge.Cuts") (width 0.1) (fill none))
-  (gr_circle (center 181.76875 -143.66875) (end 181.76875 -145.25625) (layer "Edge.Cuts") (width 0.1) (fill none))
-  (gr_circle (center -77.7875 -90.4875) (end -77.7875 -92.075) (layer "Edge.Cuts") (width 0.1) (fill none))
+  (gr_circle (center -3.175 -143.66875) (end -2.38125 -143.66875) (layer "Edge.Cuts") (width 0.1) (fill none))
+  (gr_circle (center 145.25625 -128.5875) (end 145.25625 -129.38125) (layer "Edge.Cuts") (width 0.1) (fill none))
+  (gr_circle (center -150.01875 -46.83125) (end -149.225 -47.625) (layer "Edge.Cuts") (width 0.1) (fill none))
+  (gr_circle (center 181.76875 -143.66875) (end 181.76875 -144.4625) (layer "Edge.Cuts") (width 0.1) (fill none))
+  (gr_circle (center -77.7875 -90.4875) (end -77.7875 -91.28125) (layer "Edge.Cuts") (width 0.1) (fill none))
   (segment (start -129.921 -89.408) (end -129.29425 -88.78125) (width 0.381) (layer "F.Cu") (net 1))
   (segment (start -129.921 -92.71) (end -129.921 -89.408) (width 0.381) (layer "F.Cu") (net 1))
@@
   (segment (start 14.12875 -141.72875) (end 14.12875 -140.82875) (width 0.254) (layer "B.Cu") (net 100))
   (segment (start -125.095 -109.347) (end -125.095 -109.3115) (width 0.254) (layer "B.Cu") (net 100))
-  (zone (net 0) (net_name "") (layer "B.Cu") (hatch edge 0.508)
+  (zone (net 2) (net_name "GND") (layer "B.Cu") (hatch edge 0.508)
     (connect_pads (clearance 0.508))
     (min_thickness 0.254) (filled_areas_thickness no)
@@
       (pts
         (xy -107.95 -42.8625)
-        (xy -153.9875 -42.8625)
+        (xy -154.78125 -42.8625)
         (xy -153.9875 -147.6375)
         (xy -107.95 -147.6375)
       )
     )
+  )
+  (zone (net 2) (net_name "GND") (layer "B.Cu") (hatch edge 0.508)
+    (connect_pads (clearance 0.508))
+    (min_thickness 0.254) (filled_areas_thickness no)
+    (fill yes (thermal_gap 0.508) (thermal_bridge_width 0.508))
+    (polygon
+      (pts
+        (xy 185.7375 -42.8625)
+        (xy 175.41875 -42.8625)
+        (xy 175.41875 -147.6375)
+        (xy 185.7375 -147.6375)
+      )
+    )
