File: Function Keys/Function Keys PCB/Function Keys PCB.kicad_pcb (KiCad board)
At the start: 2 copper layers, 30 parts, among them J1 Conn_01x05_Female, J2 Conn_01x05_Male

Commit message: Started placement / wiring
Parts:
- removed J2: Conn_01x05_Male, Connector_JST:JST_PH_B5B-PH-K_1x05_P2.00mm_Vertical
- removed R1, R2: 100, Resistor_SMD:R_0805_2012Metric
- J1: value Conn_01x05_Female -> Conn_01x18_Male; footprint Connector_JST:JST_PH_B5B-PH-K_1x05_P2.00mm_Vertical -> Connector_JST:JST_SH_SM20B-SRSS-TB_1x20-1MP_P1.00mm_Horizontal
- moved J1 25.8 mm to (146.8, 73.0), turned to 180 degrees
Connections:
- D1 pad 1: ROW0 -> ROW10
- D10 pad 1: ROW0 -> ROW10
- D11 pad 1: ROW0 -> ROW10
- D12 pad 1: ROW0 -> ROW10
- D13 pad 1: ROW0 -> ROW10
- D2 pad 1: ROW0 -> ROW10
- D3 pad 1: ROW0 -> ROW10
- D4 pad 1: ROW0 -> ROW10
- D5 pad 1: ROW0 -> ROW10
- D6 pad 1: ROW0 -> ROW10
- D7 pad 1: ROW0 -> ROW10
- D8 pad 1: ROW0 -> ROW10
- D9 pad 1: ROW0 -> ROW10
- J1 pad 3: Net-(J1-Pad3) -> COL0
- J1 pad 4: unconnected-(J1-Pad4) -> COL1
- J1 pad 5: GND -> COL2
Routing:
- net ROW10: track 0.00 -> 350.9 mm
- net ROW0: track 261.5 -> 0.00 mm

Commit message: Finished wiring / placement
Routing:
- net COL0: track 0.00 -> 143.0 mm, vias 0 -> 12
- net COL12: track 0.00 -> 130.4 mm, vias 0 -> 8
- net COL1: track 0.00 -> 123.0 mm, vias 0 -> 10
- net COL11: track 0.00 -> 112.4 mm, vias 0 -> 6
- net COL2: track 0.00 -> 103.2 mm, vias 0 -> 8
- net COL10: track 0.00 -> 92.5 mm, vias 0 -> 4
- net COL3: track 0.00 -> 83.1 mm, vias 0 -> 6
- net COL9: track 0.00 -> 72.3 mm, vias 0 -> 2
- net COL4: track 0.00 -> 63.0 mm, vias 0 -> 4
- net COL8: track 0.00 -> 52.6 mm, vias 0 -> 2
- net COL5: track 0.00 -> 43.0 mm, vias 0 -> 2
- net COL7: track 0.00 -> 40.0 mm
- net COL6: track 0.00 -> 22.9 mm, vias 0 -> 2
- net ROW10: track 350.9 -> 368.4 mm, vias 0 -> 2
Other:
- board outline added: 247.6 x 26.2 mm

Commit message: Added ground fill
Routing:
- added copper zone on B.Cu, net GND
Changed lines of the file:
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@@
   (segment (start 201.6125 73.025) (end 198.4375 73.025) (width 0.25) (layer "B.Cu") (net 28))
   (segment (start 160.3375 72.23125) (end 199.23125 72.23125) (width 0.25) (layer "F.Cu") (net 29))
-  (segment (start 220.6625 72.23125) (end 219.953586 72.23125) (width 0.25) (layer "F.Cu") (net 29))
-  (segment (start 238.28375 56.99125) (end 238.28375 70.485) (width 0.25) (layer "F.Cu") (net 29))
+  (segment (start 238.28375 71.27875) (end 238.28375 56.99125) (width 0.25) (layer "F.Cu") (net 29))
+  (segment (start 237.33125 72.23125) (end 238.28375 71.27875) (width 0.25) (layer "F.Cu") (net 29))
+  (segment (start 219.936619 72.248217) (end 219.953586 72.23125) (width 0.25) (layer "F.Cu") (net 29))
   (segment (start 143.34375 72.55625) (end 143.66875 72.23125) (width 0.25) (layer "F.Cu") (net 29))
-  (segment (start 238.28375 70.485) (end 238.28375 70.64375) (width 0.25) (layer "F.Cu") (net 29))
-  (segment (start 237.33125 72.23125) (end 220.6625 72.23125) (width 0.25) (layer "F.Cu") (net 29))
-  (segment (start 238.28375 71.27875) (end 237.33125 72.23125) (width 0.25) (layer "F.Cu") (net 29))
-  (segment (start 238.28375 70.485) (end 238.28375 71.27875) (width 0.25) (layer "F.Cu") (net 29))
   (segment (start 143.34375 75.025) (end 143.34375 72.55625) (width 0.25) (layer "F.Cu") (net 29))
+  (segment (start 219.953586 72.23125) (end 237.33125 72.23125) (width 0.25) (layer "F.Cu") (net 29))
   (segment (start 217.4875 72.23125) (end 200.90825 72.23125) (width 0.25) (layer "F.Cu") (net 29))
-  (segment (start 219.953586 72.23125) (end 219.936619 72.248217) (width 0.25) (layer "F.Cu") (net 29))
   (via (at 143.66875 72.23125) (size 0.8) (drill 0.4) (layers "F.Cu" "B.Cu") (net 29))
   (via (at 199.23125 72.23125) (size 0.8) (drill 0.4) (layers "F.Cu" "B.Cu") (net 29))
@@
   (segment (start 125.16425 62.79575) (end 122.99375 62.79575) (width 0.25) (layer "B.Cu") (net 31))
   (segment (start 67.818 62.738) (end 65.786 62.738) (width 0.25) (layer "B.Cu") (net 31))
+  (zone (net 18) (net_name "GND") (layer "B.Cu") (hatch edge 0.508)
+    (connect_pads (clearance 0.508))
+    (min_thickness 0.254) (filled_areas_thickness no)
+    (fill yes (thermal_gap 0.508) (thermal_bridge_width 0.508))
+    (polygon
+      (pts
+        (xy 270.66875 76.2)
+        (xy 23.01875 76.2)
+        (xy 23.01875 69.05625)
+        (xy 270.66875 69.05625)
+      )
+    )
+  )
 )
