File: Function Keys/Function Keys PCB/Function Keys PCB.kicad_pcb (KiCad board)
At the start: 2 copper layers, 247.6 x 26.2 mm, 27 parts, among them J1 Conn_01x18_Male

Commit message: Updated connectors and added through holes
Parts:
- J1: value Conn_01x18_Male -> Conn_02x10_Counter_Clockwise; footprint Connector_JST:JST_SH_SM20B-SRSS-TB_1x20-1MP_P1.00mm_Horizontal -> Connector_PinHeader_2.54mm:PinHeader_2x10_P2.54mm_Horizontal
- moved J1 11.5 mm to (158.3, 72.1), turned to -90 degrees
Connections:
- J1 pad 19: (no net) -> unconnected-(J1-Pad19)
- J1 pad 20: (no net) -> unconnected-(J1-Pad20)
Routing:
- net COL7: track 40.0 -> 34.0 mm
- net ROW10: track 368.4 -> 363.1 mm
- net COL11: track 112.2 -> 115.6 mm, vias 6 -> 0
- net COL6: track 22.9 -> 20.0 mm
- net COL9: track 72.3 -> 74.9 mm
- net COL8: track 52.6 -> 50.4 mm
- net COL4: track 63.0 -> 60.8 mm
- net COL2: track 103.2 -> 101.1 mm
- net COL12: track 130.4 -> 132.3 mm, vias 8 -> 6
- net COL1: track 123.0 -> 124.9 mm
- net COL10: track 92.5 -> 90.9 mm
- net COL3: track 83.1 -> 84.2 mm
- net COL0: track 143.0 -> 141.9 mm
- net COL5: track 43.0 -> 43.6 mm
Other:
- outline, holes or cut-outs redrawn
