File: Function Keys/Function Keys PCB/Function Keys PCB.kicad_pcb (KiCad board)
At the start: 2 copper layers, 247.6 x 26.2 mm, 27 parts, among them J1 Conn_02x10_Counter_Clockwise

Commit message: Lengthened board & moved ground pin
Connections:
- J1 pad 18: GND -> unconnected-(J1-Pad18)
- J1 pad 19: unconnected-(J1-Pad19) -> GND
Other:
- board size 247.6 x 26.2 mm -> 247.6 x 28.6 mm
Changed lines of the file:
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@@
   (net 30 "COL12")
   (net 31 "COL0")
-  (net 32 "unconnected-(J1-Pad19)")
+  (net 32 "unconnected-(J1-Pad18)")
   (net 33 "unconnected-(J1-Pad20)")
   (footprint "MX_Alps_Hybrid:MX-1U-NoLED" (layer "F.Cu")
@@
       (net 1 "ROW10") (pinfunction "Pin_17") (pintype "passive"))
     (pad "18" thru_hole oval (at 2.54 20.32 270) (size 1.7 1.7) (drill 1) (layers *.Cu *.Mask)
-      (net 18 "GND") (pinfunction "Pin_18") (pintype "passive"))
+      (net 32 "unconnected-(J1-Pad18)") (pinfunction "Pin_18") (pintype "passive"))
     (pad "19" thru_hole oval (at 0 22.86 270) (size 1.7 1.7) (drill 1) (layers *.Cu *.Mask)
-      (net 32 "unconnected-(J1-Pad19)") (pinfunction "Pin_19") (pintype "passive"))
+      (net 18 "GND") (pinfunction "Pin_19") (pintype "passive"))
     (pad "20" thru_hole oval (at 2.54 22.86 270) (size 1.7 1.7) (drill 1) (layers *.Cu *.Mask)
       (net 33 "unconnected-(J1-Pad20)") (pinfunction "Pin_20") (pintype "passive"))
@@
   )
   (gr_circle (center 71.4375 72.23125) (end 71.4375 71.4375) (layer "Edge.Cuts") (width 0.1) (fill none))
-  (gr_line (start 268.2875 76.2) (end 25.4 76.2) (layer "Edge.Cuts") (width 0.15))
+  (gr_line (start 268.2875 78.58125) (end 25.4 78.58125) (layer "Edge.Cuts") (width 0.15))
   (gr_circle (center 203.99375 51.59375) (end 203.99375 50.8) (layer "Edge.Cuts") (width 0.1) (fill none))
-  (gr_arc (start 270.66875 73.81875) (mid 269.971298 75.502548) (end 268.2875 76.2) (layer "Edge.Cuts") (width 0.15))
-  (gr_arc (start 25.4 76.2) (mid 23.716202 75.502548) (end 23.01875 73.81875) (layer "Edge.Cuts") (width 0.15))
   (gr_arc (start 23.01875 52.3875) (mid 23.716202 50.703702) (end 25.4 50.00625) (layer "Edge.Cuts") (width 0.15))
   (gr_circle (center 146.84375 51.59375) (end 146.84375 50.8) (layer "Edge.Cuts") (width 0.1) (fill none))
@@
   (gr_circle (center 89.69375 51.59375) (end 89.69375 50.8) (layer "Edge.Cuts") (width 0.1) (fill none))
   (gr_circle (center 261.14375 72.23125) (end 261.14375 71.4375) (layer "Edge.Cuts") (width 0.1) (fill none))
-  (gr_line (start 23.01875 73.81875) (end 23.01875 52.3875) (layer "Edge.Cuts") (width 0.15))
+  (gr_arc (start 25.4 78.58125) (mid 23.716202 77.883798) (end 23.01875 76.2) (layer "Edge.Cuts") (width 0.15))
+  (gr_line (start 23.01875 76.2) (end 23.01875 52.3875) (layer "Edge.Cuts") (width 0.15))
   (gr_circle (center 31.75 51.59375) (end 31.75 50.8) (layer "Edge.Cuts") (width 0.1) (fill none))
-  (gr_line (start 270.66875 73.81875) (end 270.66875 52.3875) (layer "Edge.Cuts") (width 0.15))
+  (gr_line (start 270.66875 76.2) (end 270.66875 52.3875) (layer "Edge.Cuts") (width 0.15))
   (gr_circle (center 223.04375 72.23125) (end 223.04375 71.4375) (layer "Edge.Cuts") (width 0.1) (fill none))
+  (gr_arc (start 270.66875 76.2) (mid 269.971298 77.883798) (end 268.2875 78.58125) (layer "Edge.Cuts") (width 0.15))
   (segment (start 40.48125 61.18125) (end 41.43475 61.18125) (width 0.25) (layer "F.Cu") (net 1))
   (segment (start 79.883 60.833) (end 79.883 53.086) (width 0.25) (layer "F.Cu") (net 1))
@@
     (polygon
       (pts
-        (xy 270.66875 76.2)
-        (xy 160.3375 76.2)
+        (xy 270.66875 78.58125)
+        (xy 160.3375 78.58125)
         (xy 160.3375 69.05625)
         (xy 270.66875 69.05625)
@@
     (polygon
       (pts
-        (xy 132.55625 76.2)
-        (xy 23.01875 76.2)
+        (xy 132.55625 78.58125)
+        (xy 23.01875 78.58125)
         (xy 23.01875 69.05625)
         (xy 132.55625 69.05625)
