File: Navigation Keys/Navigation Keys.kicad_pcb (KiCad board)
At the start: 2 copper layers, 73.8 x 76.2 mm, 22 parts, among them J1 Conn_01x19_Female, J2 Conn_01x19_Male

Commit message: Updated connectors + added mounting holes
Parts:
- J1: value Conn_01x19_Female -> Conn_02x10_Counter_Clockwise; footprint Connector_JST:JST_SH_SM20B-SRSS-TB_1x20-1MP_P1.00mm_Horizontal -> Connector_PinSocket_2.54mm:PinSocket_2x10_P2.54mm_Horizontal
- J2: value Conn_01x19_Male -> Conn_02x10_Counter_Clockwise; footprint Connector_JST:JST_SH_SM20B-SRSS-TB_1x20-1MP_P1.00mm_Horizontal -> Connector_PinHeader_2.54mm:PinHeader_2x10_P2.54mm_Horizontal
- moved J2 13.2 mm to (211.9, 88.1), turned to 0 degrees
- moved J1 13.1 mm to (132.6, 87.8), turned to 0 degrees
Connections:
- J1 pad 20: (no net) -> unconnected-(J1-Pad20)
- J2 pad 20: (no net) -> unconnected-(J2-Pad20)
Routing:
- net COL7: track 72.0 -> 117.8 mm, vias 8 -> 6
- net COL9: track 72.6 -> 114.5 mm
- net COL6: track 74.3 -> 106.1 mm, vias 8 -> 6
- net ROW5: track 127.3 -> 151.9 mm, vias 10 -> 8
- net COL1: track 143.1 -> 167.1 mm, vias 6 -> 4
- net ROW6: track 92.9 -> 113.4 mm, vias 8 -> 10
- net COL3: track 148.1 -> 168.1 mm, vias 6 -> 4
- net COL5: track 92.5 -> 112.2 mm, vias 8 -> 6
- net COL2: track 143.3 -> 161.8 mm, vias 8 -> 4
- net ROW8: track 146.7 -> 134.7 mm, vias 2 -> 4
- net COL4: track 94.4 -> 105.3 mm, vias 8 -> 6
- net COL8: track 70.3 -> 79.4 mm
- net COL10: track 73.4 -> 82.2 mm
- net COL0: track 108.1 -> 102.8 mm, vias 10 -> 6
- net ROW9: track 83.4 -> 88.4 mm, vias 8 -> 4
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Other:
- board size 73.8 x 76.2 mm -> 87.3 x 76.2 mm

Commit message: Extended pcb for connectors
Other:
- board size 87.3 x 76.2 mm -> 92.1 x 76.2 mm
Changed lines of the file:
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@@
       (net 11 "Net-(D7-Pad2)") (pinfunction "ROW") (pintype "passive"))
   )
-  (gr_arc (start 215.9 134.9375) (mid 215.202548 136.621298) (end 213.51875 137.31875) (layer "Edge.Cuts") (width 0.15))
-  (gr_arc (start 128.5875 63.5) (mid 129.284952 61.816202) (end 130.96875 61.11875) (layer "Edge.Cuts") (width 0.15))
-  (gr_line (start 215.9 63.5) (end 215.9 134.9375) (layer "Edge.Cuts") (width 0.15))
+  (gr_arc (start 128.5875 137.31875) (mid 126.903702 136.621298) (end 126.20625 134.9375) (layer "Edge.Cuts") (width 0.15))
+  (gr_line (start 218.28125 63.5) (end 218.28125 134.9375) (layer "Edge.Cuts") (width 0.15))
   (gr_circle (center 132.55625 133.35) (end 132.55625 132.55625) (layer "Edge.Cuts") (width 0.1) (fill none))
+  (gr_arc (start 126.20625 63.5) (mid 126.903702 61.816202) (end 128.5875 61.11875) (layer "Edge.Cuts") (width 0.15))
   (gr_circle (center 191.29375 103.98125) (end 191.29375 103.1875) (layer "Edge.Cuts") (width 0.1) (fill none))
   (gr_circle (center 211.93125 133.35) (end 212.725 133.35) (layer "Edge.Cuts") (width 0.1) (fill none))
-  (gr_line (start 128.5875 63.5) (end 128.5875 134.9375) (layer "Edge.Cuts") (width 0.15))
-  (gr_line (start 213.51875 61.11875) (end 130.96875 61.11875) (layer "Edge.Cuts") (width 0.15))
-  (gr_arc (start 130.96875 137.31875) (mid 129.284952 136.621298) (end 128.5875 134.9375) (layer "Edge.Cuts") (width 0.15))
+  (gr_arc (start 218.28125 134.9375) (mid 217.583798 136.621298) (end 215.9 137.31875) (layer "Edge.Cuts") (width 0.15))
+  (gr_line (start 126.20625 63.5) (end 126.20625 134.9375) (layer "Edge.Cuts") (width 0.15))
+  (gr_line (start 215.9 61.11875) (end 128.5875 61.11875) (layer "Edge.Cuts") (width 0.15))
   (gr_circle (center 153.19375 115.8875) (end 153.19375 115.09375) (layer "Edge.Cuts") (width 0.1) (fill none))
   (gr_circle (center 132.55625 65.0875) (end 132.55625 64.29375) (layer "Edge.Cuts") (width 0.1) (fill none))
-  (gr_line (start 130.96875 137.31875) (end 213.51875 137.31875) (layer "Edge.Cuts") (width 0.15))
+  (gr_arc (start 215.9 61.11875) (mid 217.583798 61.816202) (end 218.28125 63.5) (layer "Edge.Cuts") (width 0.15))
+  (gr_line (start 128.5875 137.31875) (end 215.9 137.31875) (layer "Edge.Cuts") (width 0.15))
   (gr_circle (center 211.93125 65.0875) (end 211.93125 64.29375) (layer "Edge.Cuts") (width 0.1) (fill none))
-  (gr_arc (start 213.51875 61.11875) (mid 215.202548 61.816202) (end 215.9 63.5) (layer "Edge.Cuts") (width 0.15))
   (segment (start 180.18125 73.81875) (end 180.18125 72.29375) (width 0.25) (layer "F.Cu") (net 1))
   (segment (start 204.65 74.68175) (end 204.58075 74.6125) (width 0.25) (layer "F.Cu") (net 1))
@@
     (polygon
       (pts
-        (xy 215.9 137.31875)
+        (xy 218.28125 137.31875)
         (xy 200.81875 137.31875)
         (xy 200.81875 61.11875)
-        (xy 215.9 61.11875)
+        (xy 218.28125 61.11875)
       )
     )
@@
       (pts
         (xy 143.66875 137.31875)
-        (xy 128.5875 137.31875)
-        (xy 128.5875 61.11875)
+        (xy 126.20625 137.31875)
+        (xy 126.20625 61.11875)
         (xy 143.66875 61.11875)
       )
